File: pcb/main_pcb_project/main_pcb_project.kicad_sch (KiCad schematic)
At the start: 0 parts

Commit message: Add our names to the schematic title block
Other:
- company: (none) -> RoboCup
- title: (none) -> Double Krish Main PCB Design
Changed lines of the file:
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@@
 	(generator_version "10.0")
 	(paper "A4")
+	(title_block
+		(title "Double Krish Main PCB Design")
+		(company "RoboCup")
+	)
 	(sheet_instances
 		(path "/"
