File: pcb/main_pcb_project/main_pcb_project.kicad_sch (KiCad schematic)
At the start: 0 parts

Commit message: Added hierarchical sheet for microcontroller
Other:
- added sheet RP2040 Microcontroller (untitled.kicad_sch)
Changed lines of the file:
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@@
 		(comment 1 "Garrett Coker")
+	)
+	(sheet
+		(at 118.11 26.67)
+		(size 53.34 48.26)
+		(exclude_from_sim no)
+		(in_bom yes)
+		(on_board yes)
+		(dnp no)
+		(fields_autoplaced yes)
+		(stroke
+			(width 0.1524)
+			(type solid)
+		)
+		(fill
+			(color 0 0 0 0)
+		)
+		(property "Sheetname" "RP2040 Microcontroller"
+			(at 118.11 25.9584 0)
+			(show_name no)
+			(do_not_autoplace no)
+			(effects
+				(font
+					(size 1.27 1.27)
+				)
+				(justify left bottom)
+			)
+		)
+		(property "Sheetfile" "untitled.kicad_sch"
+			(at 118.11 75.5146 0)
+			(show_name no)
+			(do_not_autoplace no)
+			(effects
+				(font
+					(size 1.27 1.27)
+				)
+				(justify left top)
+			)
+		)
+		(instances
+			(project "main_pcb_project"
+				(path "/9164435f-a95c-403a-a8b4-52de8af1bdc8"
+					(page "2")
+				)
+			)
+		)
 	)
 	(sheet_instances
