File: pcb/main_pcb_project/untitled.kicad_sch (KiCad schematic)
At the start: 1 part, among them U1 RP2040

Commit message: Continued RP2040 implementation
Parts:
- removed U1: RP2040, Package_DFN_QFN:QFN-56-1EP_7x7mm_P0.4mm_EP3.2x3.2mm, symbol MCU_RaspberryPi:RP2040
Other:
- company: (none) -> Double Krish
- title: (none) -> RP2040 Implementation
Changed lines of the file:
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@@
 	(generator_version "10.0")
 	(paper "A4")
-	(symbol
-		(lib_id "MCU_RaspberryPi:RP2040")
-		(at 139.7 102.87 0)
-		(unit 1)
-		(body_style 1)
-		(exclude_from_sim no)
-		(in_bom yes)
-		(on_board yes)
-		(in_pos_files yes)
-		(dnp no)
-		(fields_autoplaced yes)
-		(property "Reference" "U1"
-			(at 141.8433 147.32 0)
-			(show_name no)
-			(do_not_autoplace no)
-			(effects
-				(font
-					(size 1.27 1.27)
-				)
-				(justify left)
-			)
-		)
-		(property "Value" "RP2040"
-			(at 141.8433 149.86 0)
-			(show_name no)
-			(do_not_autoplace no)
-			(effects
-				(font
-					(size 1.27 1.27)
-				)
-				(justify left)
-			)
-		)
-		(property "Footprint" "Package_DFN_QFN:QFN-56-1EP_7x7mm_P0.4mm_EP3.2x3.2mm"
-			(at 139.7 102.87 0)
-			(hide yes)
-			(show_name no)
-			(do_not_autoplace no)
-			(effects
-				(font
-					(size 1.27 1.27)
-				)
-			)
-		)
-		(property "Datasheet" "https://datasheets.raspberrypi.com/rp2040/rp2040-datasheet.pdf"
-			(at 139.7 102.87 0)
-			(hide yes)
-			(show_name no)
-			(do_not_autoplace no)
-			(effects
-				(font
-					(size 1.27 1.27)
-				)
-			)
-		)
-		(property "Description" "A microcontroller by Raspberry Pi, Dual ARM Cortex-M0+, 133MHz, no flash, 264KB SRAM, 8 PIO state machines, VQFN-56"
-			(at 139.7 102.87 0)
-			(hide yes)
-			(show_name no)
-			(do_not_autoplace no)
-			(effects
-				(font
-					(size 1.27 1.27)
-				)
-			)
-		)
-		(property private "KLC_S4.2_DVDD" "Not a standalone power converter; internal on-chip voltage regulator for digital core supply; DVDD is the digital core power supply, should be placed next to voltage regulator output."
-			(at 139.7 105.41 0)
-			(hide yes)
-			(show_name yes)
-			(do_not_autoplace no)
-			(effects
-				(font
-					(size 1.27 1.27)
-				)
-			)
-		)
-		(property private "KLC_S4.2_VREG_VOUT" "Should be placed next to DVDD."
-			(at 139.7 105.41 0)
-			(hide yes)
-			(show_name yes)
-			(do_not_autoplace no)
-			(effects
-				(font
-					(size 1.27 1.27)
-				)
-			)
-		)
-		(pin "5"
-		)
-		(pin "10"
-		)
-		(pin "11"
-		)
-		(pin "9"
-		)
-		(pin "2"
-		)
-		(pin "3"
-		)
-		(pin "4"
-		)
-		(pin "1"
-		)
-		(pin "7"
-		)
-		(pin "8"
-		)
-		(pin "6"
-		)
-		(pin "18"
-		)
-		(pin "24"
-		)
-		(pin "29"
-		)
-		(pin "30"
-		)
-		(pin "39"
-		)
-		(pin "21"
-		)
-		(pin "33"
-		)
-		(pin "19"
-		)
-		(pin "31"
-		)
-		(pin "38"
-		)
-		(pin "14"
-		)
-		(pin "34"
-		)
-		(pin "42"
-		)
-		(pin "22"
-		)
-		(pin "13"
-		)
-		(pin "23"
-		)
-		(pin "28"
-		)
-		(pin "20"
-		)
-		(pin "12"
-		)
-		(pin "27"
-		)
-		(pin "32"
-		)
-		(pin "35"
-		)
-		(pin "37"
-		)
-		(pin "41"
-		)
-		(pin "26"
-		)
-		(pin "17"
-		)
-		(pin "15"
-		)
-		(pin "36"
-		)
-		(pin "16"
-		)
-		(pin "25"
-		)
-		(pin "40"
-		)
-		(pin "43"
-		)
-		(pin "56"
-		)
-		(pin "55"
-		)
-		(pin "44"
-		)
-		(pin "46"
-		)
-		(pin "52"
-		)
-		(pin "53"
-		)
-		(pin "49"
-		)
-		(pin "57"
-		)
-		(pin "47"
-		)
-		(pin "54"
-		)
-		(pin "45"
-		)
-		(pin "50"
-		)
-		(pin "51"
-		)
-		(pin "48"
-		)
-		(instances
-			(project "main_pcb_project"
-				(path "/9164435f-a95c-403a-a8b4-52de8af1bdc8/43d08942-0182-4d4a-9589-a975afa41050"
-					(reference "U1")
-					(unit 1)
-				)
-			)
-		)
+	(title_block
+		(title "RP2040 Implementation")
+		(rev "v.0.1")
+		(company "Double Krish")
+		(comment 1 "Garrett Coker")
 	)
 )
