File: pcb/RP2040_microcontroller/RP2040_microcontroller.kicad_sch (KiCad schematic)
At the start: 0 parts

Commit message: add added in the rp2040 to the microncontroller file
Parts:
- added U1: RP2040, Package_DFN_QFN:QFN-56-1EP_7x7mm_P0.4mm_EP3.2x3.2mm, symbol MCU_RaspberryPi:RP2040
Connections:
- new net: U1.1 (IOVDD), U1.10 (IOVDD), U1.22 (IOVDD), U1.33 (IOVDD), U1.42 (IOVDD), U1.49 (IOVDD)
- new net: U1.23 (DVDD), U1.50 (DVDD)
Changed lines of the file:
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@@
 	(generator_version "10.0")
 	(paper "A4")
+	(symbol
+		(lib_id "MCU_RaspberryPi:RP2040")
+		(at 143.51 107.95 0)
+		(unit 1)
+		(body_style 1)
+		(exclude_from_sim no)
+		(in_bom yes)
+		(on_board yes)
+		(in_pos_files yes)
+		(dnp no)
+		(fields_autoplaced yes)
+		(property "Reference" "U1"
+			(at 145.6533 152.4 0)
+			(show_name no)
+			(do_not_autoplace no)
+			(effects
+				(font
+					(size 1.27 1.27)
+				)
+				(justify left)
+			)
+		)
+		(property "Value" "RP2040"
+			(at 145.6533 154.94 0)
+			(show_name no)
+			(do_not_autoplace no)
+			(effects
+				(font
+					(size 1.27 1.27)
+				)
+				(justify left)
+			)
+		)
+		(property "Footprint" "Package_DFN_QFN:QFN-56-1EP_7x7mm_P0.4mm_EP3.2x3.2mm"
+			(at 143.51 107.95 0)
+			(hide yes)
+			(show_name no)
+			(do_not_autoplace no)
+			(effects
+				(font
+					(size 1.27 1.27)
+				)
+			)
+		)
+		(property "Datasheet" "https://datasheets.raspberrypi.com/rp2040/rp2040-datasheet.pdf"
+			(at 143.51 107.95 0)
+			(hide yes)
+			(show_name no)
+			(do_not_autoplace no)
+			(effects
+				(font
+					(size 1.27 1.27)
+				)
+			)
+		)
+		(property "Description" "A microcontroller by Raspberry Pi, Dual ARM Cortex-M0+, 133MHz, no flash, 264KB SRAM, 8 PIO state machines, VQFN-56"
+			(at 143.51 107.95 0)
+			(hide yes)
+			(show_name no)
+			(do_not_autoplace no)
+			(effects
+				(font
+					(size 1.27 1.27)
+				)
+			)
+		)
+		(property private "KLC_S4.2_DVDD" "Not a standalone power converter; internal on-chip voltage regulator for digital core supply; DVDD is the digital core power supply, should be placed next to voltage regulator output."
+			(at 143.51 110.49 0)
+			(hide yes)
+			(show_name yes)
+			(do_not_autoplace no)
+			(effects
+				(font
+					(size 1.27 1.27)
+				)
+			)
+		)
+		(property private "KLC_S4.2_VREG_VOUT" "Should be placed next to DVDD."
+			(at 143.51 110.49 0)
+			(hide yes)
+			(show_name yes)
+			(do_not_autoplace no)
+			(effects
+				(font
+					(size 1.27 1.27)
+				)
+			)
+		)
+		(pin "4"
+		)
+		(pin "9"
+		)
+		(pin "5"
+		)
+		(pin "21"
+		)
+		(pin "19"
+		)
+		(pin "16"
+		)
+		(pin "11"
+		)
+		(pin "20"
+		)
+		(pin "12"
+		)
+		(pin "7"
+		)
+		(pin "8"
+		)
+		(pin "18"
+		)
+		(pin "10"
+		)
+		(pin "14"
+		)
+		(pin "15"
+		)
+		(pin "2"
+		)
+		(pin "6"
+		)
+		(pin "17"
+		)
+		(pin "1"
+		)
+		(pin "23"
+		)
+		(pin "13"
+		)
+		(pin "24"
+		)
+		(pin "22"
+		)
+		(pin "3"
+		)
+		(pin "43"
+		)
+		(pin "37"
+		)
+		(pin "52"
+		)
+		(pin "29"
+		)
+		(pin "46"
+		)
+		(pin "49"
+		)
+		(pin "47"
+		)
+		(pin "31"
+		)
+		(pin "39"
+		)
+		(pin "26"
+		)
+		(pin "40"
+		)
+		(pin "36"
+		)
+		(pin "33"
+		)
+		(pin "27"
+		)
+		(pin "34"
+		)
+		(pin "42"
+		)
+		(pin "35"
+		)
+		(pin "45"
+		)
+		(pin "32"
+		)
+		(pin "30"
+		)
+		(pin "38"
+		)
+		(pin "50"
+		)
+		(pin "53"
+		)
+		(pin "51"
+		)
+		(pin "41"
+		)
+		(pin "44"
+		)
+		(pin "25"
+		)
+		(pin "28"
+		)
+		(pin "48"
+		)
+		(pin "54"
+		)
+		(pin "55"
+		)
+		(pin "56"
+		)
+		(pin "57"
+		)
+		(instances
+			(project "RP2040_microcontroller"
+				(path "/d535c0e3-c6d0-4685-ac3f-9630a6728c77"
+					(reference "U1")
+					(unit 1)
+				)
+			)
+		)
+	)
 	(sheet_instances
 		(path "/"
