File: pcb/I2C_kicad/GPIOexpander.kicad_sch (KiCad schematic)
At the start: 0 parts

Commit message: I worked on the color sensor and also the gpio expander. I added the pull ups for the SDA and SCL on the color sensor so no need to add any more. Just put do not populate for the other I2c devices
Parts:
- added C3: 100nF, Capacitor_SMD:C_0603_1608Metric, symbol Device:C
- added R3, R4: 10kΩ, Resistor_SMD:R_0603_1608Metric, symbol Device:R
- added RN1, RN2: 10kΩ, Resistor_SMD:R_Array_Convex_4x0603, symbol Device:R_Pack04
- added SW1: SW_DIP_x08, Button_Switch_THT:SW_DIP_SPSTx08_Slide_9.78x22.5mm_W7.62mm_P2.54mm, symbol Switch:SW_DIP_x08
- added U3: TCA9534, Package_SO:TSSOP-16_4.4x5mm_P0.65mm, symbol Interface_Expansion:TCA9534
Connections:
- new net +3V3: C3.1, R3.1, R4.1, RN1.5 (R4.2), RN1.6 (R3.2), RN1.7 (R2.2), RN1.8 (R1.2), RN2.5 (R4.2), RN2.6 (R3.2), RN2.7 (R2.2), RN2.8 (R1.2), U3.16 (VDD)
- new net EXP_P0: RN1.1 (R1.1), SW1.1, U3.4 (P0)
- new net EXP_P1: RN1.2 (R2.1), SW1.2, U3.5 (P1)
- new net EXP_P2: RN1.3 (R3.1), SW1.3, U3.6 (P2)
- new net EXP_P3: RN1.4 (R4.1), SW1.4, U3.7 (P3)
- new net EXP_P4: RN2.1 (R1.1), SW1.5, U3.9 (P4)
- new net EXP_P5: RN2.2 (R2.1), SW1.6, U3.10 (P5)
- new net EXP_P6: RN2.3 (R3.1), SW1.7, U3.11 (P6)
- new net EXP_P7: RN2.4 (R4.1), SW1.8, U3.12 (P7)
- new net GND: C3.2, SW1.10, SW1.11, SW1.12, SW1.13, SW1.14, SW1.15, SW1.16, SW1.9, U3.1 (A0), U3.2 (A1), U3.3 (A2), U3.8 (GND)
- new net SCL: R4.2, U3.14 (SCL)
- new net SDA: R3.2, U3.15 (SDA)
- no-connect marks 0 -> 1
Other:
- note added: "Decoupling Capacitor needs to be placed close to Vdd"
- note added: "Making them do not populate because the Bus already has pull ups"
- note added: "Ti used 100k (ohm) resitor but part list has 10k. Both should work"
- company: (none) -> RoboCup
- title: (none) -> GPIO Expander

Commit message: fixed some labels
Other:
- note added: "These are pull up"
- moved on the sheet: RN1, RN2
