File: pcb/I2C_kicad/HallEffect.kicad_sch (KiCad schematic)
At the start: 0 parts

Commit message: Add IMU, Hall effect, and temp sensor sheets
Parts:
- added C6: 0.1uF, Capacitor_SMD:C_0603_1608Metric, symbol Device:C
- added U4: TMAG5273A2QDBVR, Package_TO_SOT_SMD:SOT-23-6, symbol Sensor_Magnetic:TMAG5273x2QDBV
Connections:
- new net +3V3: C6.1, U4.4 (VCC)
- new net GND: C6.2, U4.2 (GND), U4.3 (TEST), U4.5 (~{INT})
- new net SCL: U4.1 (SCL)
- new net SDA: U4.6 (SDA)
Other:
- note added: "INT unused: MCU polls over I2C instead; tied to GND per Table 4-1, firmware must set MASK_INTB = 1 (pg 4 in dada sheet)"
- note added: "Need to place this capsitor close to VCC"
- company: (none) -> RoboCup
- title: (none) -> Hall Effect
