File: pcb/I2C_kicad/TemperatureSensor.kicad_sch (KiCad schematic)
At the start: 0 parts

Commit message: Add IMU, Hall effect, and temp sensor sheets
Parts:
- added C7: 0.1uF, Capacitor_SMD:C_0603_1608Metric, symbol Device:C
- added U5: LM75ADP, Package_SO:TSSOP-8_3x3mm_P0.65mm, symbol Sensor_Temperature:LM75B
Connections:
- new net +3V3: C7.1, U5.8 (VCC)
- new net GND: C7.2, U5.4 (GND), U5.5 (A2), U5.6 (A1), U5.7 (A0)
- new net SCL: U5.2 (SCL)
- new net SDA: U5.1 (SDA)
- no-connect marks 0 -> 1
Other:
- note added: "A0-A2 are tied to GND to set the I2C address to 0x48 (Section 7.3, p. 6) (it said to not leave them floating)"
- note added: "Need to place Capacitor close to VCC"
- note added: "The OS pin is left unconnected because it is an open drain output and the MCU reads the temperature over I2C instead"
- company: (none) -> RoboCup
- title: (none) -> Temperture Sensor
