File: pcb/I2C_kicad/LEDPWMController.kicad_sch (KiCad schematic)
At the start: 0 parts

Commit message: Add IMU, Hall effect, and temp sensor sheets
Parts:
- added C8: 1 uF, Capacitor_SMD:C_0603_1608Metric, symbol Device:C
- added U6: IS31FL3254-QFLS4-TR, Package_DFN_QFN:QFN-32-1EP_4x4mm_P0.4mm_EP2.65x2.65mm, symbol IS31FL3254:IS31FL3254-QFLS4-TR
Connections:
- new net +3V3: U6.28 (VCC)
Other:
- company: (none) -> RoboCup
- title: (none) -> LED PWM Controller

Commit message: work was done
Parts:
- added C9: 0.1 uF, Capacitor_SMD:C_0603_1608Metric, symbol Device:C
- added D1, D2, D3, D4, D5, D6, D7, D8: CLMVC-FKA-CL1D1L71BB7C3C3, LED_SMD:LED_Cree-PLCC4_2x2mm_CW, symbol Device:LED_ABGR
- added R5: 6.8k, Resistor_SMD:R_0603_1608Metric, symbol Device:R
- added R6: 100k, Resistor_SMD:R_0603_1608Metric, symbol Device:R
Connections:
- net +3V3: now also C8.1, C9.1, D1.1 (A), D2.1 (A), D3.1 (A), D4.1 (A), D5.1 (A), D6.1 (A), D7.1 (A), D8.1 (A), R6.1
- net OUT1: now reaches U6.1 (OUT1_R1)
- net OUT1: now also D1.4 (RK)
- net OUT10: now reaches U6.10 (OUT10_R4)
- net OUT10: now also D4.4 (RK)
- net OUT11: now reaches U6.11 (OUT11_G4)
- net OUT11: now also D4.3 (GK)
- net OUT12: now reaches U6.12 (OUT12_B4)
- net OUT12: now also D4.2 (BK)
- net GND: now reaches U6.13 (GND)
- net GND: now also C8.2, U6.27 (AD), U6.29 (GND), U6.33 (GND), C9.2, R5.2
- net OUT13: now reaches U6.14 (OUT13_R5)
- net OUT13: now also D5.4 (RK)
- net OUT14: now reaches U6.15 (OUT14_G5)
- net OUT14: now also D5.3 (GK)
- net OUT15: now reaches U6.16 (OUT15_B5)
- net OUT15: now also D5.2 (BK)
- net OUT16: now reaches U6.17 (OUT16_R6)
- net OUT16: now also D6.4 (RK)
- net OUT17: now reaches U6.18 (OUT17_G6)
- net OUT17: now also D6.3 (GK)
- net OUT18: now reaches U6.19 (OUT18_B6)
- net OUT18: now also D6.2 (BK)
- net OUT2: now reaches U6.2 (OUT2_G1)
- net OUT2: now also D1.3 (GK)
- net OUT19: now reaches U6.20 (OUT19_R7)
- net OUT19: now also D7.4 (RK)
- net OUT20: now reaches U6.21 (OUT20_G7)
- net OUT20: now also D7.3 (GK)
- net OUT21: now reaches U6.22 (OUT21_B7)
- net OUT21: now also D7.2 (BK)
- net OUT22: now reaches U6.23 (OUT22_R8)
- net OUT22: now also D8.4 (RK)
- net OUT23: now reaches U6.24 (OUT23_G8)
- net OUT23: now also D8.3 (GK)
- net OUT24: now reaches U6.25 (OUT24_B8)
- net OUT24: now also D8.2 (BK)
- net at U6.26 (~{SDB}): now also R6.2
- net OUT3: now reaches U6.3 (OUT3_B1)
- net OUT3: now also D1.2 (BK)
- net at U6.30 (ISET): now also R5.1
- net SDA: now reaches U6.31 (SDA)
- net SCL: now reaches U6.32 (SCL)
- net OUT4: now reaches U6.4 (OUT4_R2)
- net OUT4: now also D2.4 (RK)
- net OUT5: now reaches U6.5 (OUT5_G2)
- net OUT5: now also D2.3 (GK)
- net OUT6: now reaches U6.6 (OUT6_B2)
- net OUT6: now also D2.2 (BK)
- net OUT7: now reaches U6.7 (OUT7_R3)
- net OUT7: now also D3.4 (RK)
- net OUT8: now reaches U6.8 (OUT8_G3)
- net OUT8: now also D3.3 (GK)
- net OUT9: now reaches U6.9 (OUT9_B3)
- net OUT9: now also D3.2 (BK)
Other:
- note added: "AD to GND sets I2C address 0x30 (pg 8)"
- note added: "Need to place these capcitors near Vcc"
- note added: "R_ISET = 6.8k gives a current of 11.1mA using formula on pg 17"
- note added: "SDB pulled High"
- note added: "pin 33 is the thermal pad and it says it needs to be connected to ground"
- moved on the sheet: C8, U6
