File: pcb/RP2040_mcu_kicad/RP2040_microcontroller.kicad_sch (KiCad schematic)
At the start: 18 parts, among them J1 USB_B_Micro, SW1 SW_SPST, U1 RP2040, U2 W25Q128JVS

Commit message: Finished 2040
Parts:
- added C11, C12: 10u, Capacitor_SMD:C_0402_1005Metric, symbol Device:C
- added C13, C14: 15p, Capacitor_SMD:C_0402_1005Metric, symbol Device:C
- added J2: Conn_01x03, Connector_PinHeader_2.54mm:PinHeader_1x03_P2.54mm_Vertical, symbol Connector_Generic:Conn_01x03
- added R5: 1k, Resistor_SMD:R_0402_1005Metric, symbol Device:R
- added SW2: SW_Push, SKRPABE010, symbol Switch:SW_Push
- added U3: NCP1117-3.3_SOT223, Package_TO_SOT_SMD:SOT-223-3_TabPin2, symbol Regulator_Linear:NCP1117-3.3_SOT223
- added Y1: ABM8-272-T3, 3.2x2.5mm, symbol Device:Crystal_GND24
- C10: value C -> 100n; footprint Package_DFN_QFN:QFN-56-1EP_7x7mm_P0.4mm_EP3.2x3.2mm -> Capacitor_SMD:C_0402_1005Metric
- J1: footprint (none) -> Connector_USB:USB_Micro-B_Amphenol_10118194_Horizontal
- R1, R2: footprint Package_DIP:DIP-8_W7.62mm -> Resistor_SMD:R_0402_1005Metric
- R3, R4: value R -> 27; footprint (none) -> Resistor_SMD:R_0402_1005Metric
- SW1: value SW_SPST -> SW_Push; footprint Button_Switch_SMD:Nidec_Copal_CAS-120A -> SKRPABE010
- U2: value W25Q128JVS -> W25Q16JVUXIQ TR; footprint Package_SO:SOIC-8_5.3x5.3mm_P1.27mm -> USON-8-EP (2 x 3 mm)
Connections:
- net +3V3: now also C12.1, U3.2 (VO)
- net GND: now also U1.19 (TESTEN), C11.2, C12.2, C13.1, C14.1, J2.2 (Pin_2), SW2.1, U3.1 (GND), Y1.2 (G), Y1.4 (G)
- net XIN: now reaches U1.20 (XIN)
- net XIN: now also C13.2, Y1.1
- net XOUT: now reaches U1.21 (XOUT)
- net XOUT: now also R5.2
- net at U1.24 (SWCLK): now also J2.1 (Pin_1)
- net at U1.25 (SWDIO): now also J2.3 (Pin_3)
- net at U1.26 (RUN): now also SW2.2
- net at J1.1 (VBUS): now also C11.1, U3.3 (VI)
- new net: C14.2, R5.1, Y1.3
- no-connect marks 1 -> 31
Other:
- note added: "Crystal"
