File: pcb/main_pcb_kicad/ColorSensor.kicad_sch (KiCad schematic)
At the start: 4 parts, among them U6 VEML3328

Commit message: i fixed the layout on the MCU for SDA and SCL also added page information on the subsheets
Other:
- note added: "NEED TO PUT PULL UP RESISTORS NEAR THE MCU"
- company: (none) -> RoboCup
- title: (none) -> Color Sensor
Changed lines of the file:
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@@
 	(generator_version "10.0")
 	(paper "A4")
+	(title_block
+		(title "Color Sensor")
+		(company "RoboCup")
+	)
 	(text "Place the Capsitor close to Vdd"
 		(exclude_from_sim no)
@@
 			)
 		)
+	)
+	(text "NEED TO PUT PULL UP RESISTORS \nNEAR THE MCU"
+		(exclude_from_sim no)
+		(at 138.43 128.27 0)
+		(effects
+			(font
+				(size 2.54 2.54)
+			)
+		)
