File: pcb/main_pcb_kicad/GPIOexpander.kicad_sch (KiCad schematic)
At the start: 7 parts, among them SW3 SW_DIP_x08, U8 TCA9534

Commit message: i fixed the layout on the MCU for SDA and SCL also added page information on the subsheets
Other:
- company: (none) -> RoboCup
- title: (none) -> GPIO expander
Changed lines of the file:
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@@
 	(generator_version "10.0")
 	(paper "A4")
+	(title_block
+		(title "GPIO expander")
+		(company "RoboCup")
+	)
 	(text "Decoupling Capacitor needs \nto be placed close to Vdd"
 		(exclude_from_sim no)
