File: pcb/main_pcb_kicad/HallEffect.kicad_sch (KiCad schematic)
At the start: 2 parts, among them U5 TMAG5273A2QDBVR

Commit message: i fixed the layout on the MCU for SDA and SCL also added page information on the subsheets
Other:
- company: (none) -> RoboCup
- title: (none) -> Hall Effect
Changed lines of the file:
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@@
 	(generator_version "10.0")
 	(paper "A4")
+	(title_block
+		(title "Hall Effect")
+		(company "RoboCup")
+	)
 	(text "INT unused: MCU polls over I2C instead; \ntied to GND per Table 4-1, \nfirmware must set MASK_INTB = 1\n(pg 4 in dada sheet)"
 		(exclude_from_sim no)
