File: pcb/main_pcb_kicad/IMU.kicad_sch (KiCad schematic)
At the start: 4 parts, among them U4 ICM-42605

Commit message: i fixed the layout on the MCU for SDA and SCL also added page information on the subsheets
Other:
- company: (none) -> RoboCUp
- title: (none) -> IMU
Changed lines of the file:
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@@
 	(generator_version "10.0")
 	(paper "A4")
+	(title_block
+		(title "IMU")
+		(company "RoboCUp")
+	)
 	(junction
 		(at 68.58 96.52)
