File: pcb/main_pcb_kicad/LEDPWMController.kicad_sch (KiCad schematic)
At the start: 13 parts, among them U9 IS31FL3254-QFLS4-TR

Commit message: i fixed the layout on the MCU for SDA and SCL also added page information on the subsheets
Other:
- company: (none) -> RoboCup
- title: (none) -> LED PWM Controller
Changed lines of the file:
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@@
 	(generator_version "10.0")
 	(paper "A4")
+	(title_block
+		(title "LED PWM Controller")
+		(company "RoboCup")
+	)
 	(text "Need to place these capcitors\nnear Vcc"
 		(exclude_from_sim no)
