File: pcb/main_pcb_kicad/TemperatureSensor.kicad_sch (KiCad schematic)
At the start: 2 parts, among them U7 LM75ADP

Commit message: i fixed the layout on the MCU for SDA and SCL also added page information on the subsheets
Other:
- company: (none) -> RoboCup
- title: (none) -> Temperature Sensor
Changed lines of the file:
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@@
 	(generator_version "10.0")
 	(paper "A4")
+	(title_block
+		(title "Temperature Sensor")
+		(company "RoboCup")
+	)
 	(text "The OS pin is left unconnected\n because it is an open drain output\n and the MCU reads the temperature over I2C instead"
 		(exclude_from_sim no)
