File: pcb/rj-electrical-training/ind_leds.kicad_sch (KiCad schematic)
At the start: 14 parts

Commit message: Integrated LEDs to circuit
Parts:
- removed D6, D7, D8, D9: RED, LED_SMD:LED_0603_1608Metric, symbol Device:LED
- removed R18, R19, R20, R21: 1k, Resistor_SMD:R_0402_1005Metric, symbol Device:R
Connections:
- net ind_led0 renamed slave_power_led
- net ind_led1 renamed usb_power_led
- net ind_led2 renamed color_sensor_led
Other:
- title: (none) -> Debug LEDs
