File: pcb/rj-electrical-training/usb_conn.kicad_sch (KiCad schematic)
At the start: 9 parts, among them J1 USB_C_Receptacle_USB2.0_16P, J2 SWD, U3 AP2112K-3.3, U4 USBLC6-2P6, U5 USBLC6-2P6

Commit message: Integrated LEDs to circuit
Changed lines of the file:
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@@
 	(rectangle
 		(start 165.1 50.8)
-		(end 215.9 88.9)
+		(end 226.06 88.9)
 		(stroke
 			(width 0)
@@
 	)
 	(junction
+		(at 203.2 62.23)
+		(diameter 0)
+		(color 0 0 0 0)
+	)
+	(junction
 		(at 102.87 72.39)
 		(diameter 0)
@@
 	(wire
 		(pts
+			(xy 205.74 62.23) (xy 203.2 62.23)
+		)
+		(stroke
+			(width 0)
+			(type default)
+		)
+	)
+	(wire
+		(pts
 			(xy 78.74 80.01) (xy 81.28 80.01)
 		)
@@
 		)
 	)
+	(hierarchical_label "usb_power_led"
+		(shape output)
+		(at 205.74 62.23 0)
+		(effects
+			(font
+				(size 1.27 1.27)
+			)
+			(justify left)
+		)
+	)
+	(hierarchical_label "usb_power_led"
+		(shape output)
+		(at 0.3048 0.8096 0)
+		(effects
+			(font
+				(size 1.27 1.27)
+			)
+			(justify left)
+		)
+	)
+	(hierarchical_label "usb_power_led"
+		(shape output)
+		(at 2.8448 3.3496 0)
+		(effects
+			(font
+				(size 1.27 1.27)
+			)
+			(justify left)
+		)
+	)
