File: pcb/mcu.kicad_sch (KiCad schematic)
At the start: 0 parts

Commit message: Add files via upload
Parts:
- added C1, C2: 1µF, Capacitor_SMD:C_0603_1608Metric, symbol Device:C
- added C10, C11, C12, C3, C4, C5, C6, C7, C8, C9: 100nF, Capacitor_SMD:C_0603_1608Metric, symbol Device:C
- added R1: 10k, Resistor_SMD:R_0603_1608Metric, symbol Device:R
- added U1: RP2040, Package_DFN_QFN:QFN-56-1EP_7x7mm_P0.4mm_EP3.2x3.2mm, symbol MCU_RaspberryPi:RP2040
Connections:
- new net: R1.2, U1.26 (RUN)
- new net +3V3: C1.1, C10.1, C3.1, C4.1, C5.1, C6.1, C7.1, C8.1, C9.1, R1.1, U1.1 (IOVDD), U1.10 (IOVDD), U1.22 (IOVDD), U1.33 (IOVDD), U1.42 (IOVDD), U1.43 (ADC_AVDD), U1.44 (VREG_VIN), U1.48 (USB_VDD), U1.49 (IOVDD)
- new net COLOR_SCL: U1.35 (GPIO23)
- new net COLOR_SDA: U1.34 (GPIO22)
- new net GND: C1.2, C10.2, C11.2, C12.2, C2.2, C3.2, C4.2, C5.2, C6.2, C7.2, C8.2, C9.2, U1.19 (TESTEN), U1.57 (GND)
- new net HALL_INT_N: U1.39 (GPIO27/ADC1)
- new net HALL_SCL: U1.32 (GPIO21)
- new net HALL_SDA: U1.31 (GPIO20)
- new net IMU_INT1: U1.38 (GPIO26/ADC0)
- new net IMU_SCL: U1.28 (GPIO17)
- new net IMU_SDA: U1.27 (GPIO16)
- new net LED_SCL: U1.37 (GPIO25)
- new net LED_SDA: U1.36 (GPIO24)
- new net LED_SDB: U1.41 (GPIO29/ADC3)
- new net SPI0_CSN: U1.3 (GPIO1)
- new net SPI0_RX: U1.2 (GPIO0)
- new net SPI0_SCK: U1.4 (GPIO2)
- new net SPI0_TX: U1.5 (GPIO3)
- new net SPI1_CSN: U1.16 (GPIO13)
- new net SPI1_RX: U1.15 (GPIO12)
- new net SPI1_SCK: U1.17 (GPIO14)
- new net SPI1_TX: U1.18 (GPIO15)
- new net TCA_INT_N: U1.14 (GPIO11)
- new net TCA_SCL: U1.7 (GPIO5)
- new net TCA_SDA: U1.6 (GPIO4)
- new net TEMP_SCL: U1.30 (GPIO19)
- new net TEMP_SDA: U1.29 (GPIO18)
- new net USER_BTN1_N: U1.8 (GPIO6)
- new net USER_BTN2_N: U1.9 (GPIO7)
- new net USER_LED1: U1.11 (GPIO8)
- new net USER_LED2: U1.12 (GPIO9)
- new net USER_LED3: U1.13 (GPIO10)
- new net VDD_CORE: C11.1, C12.1, C2.1, U1.23 (DVDD), U1.45 (VREG_VOUT), U1.50 (DVDD)
- no-connect marks 0 -> 1
Other:
- note removed: "Sheet: MCU Purpose: RP2040 core: flash, crystal, USB data, SWD, boot/reset Planned contents: - U: RP2040, decoupling per RP2040 hardware design guide - U: W25Q16JVUXIQ 2 MB QSPI flash - Y: ABM8-272-T3 12 MHz crystal + load caps - USB D+/D- with 27R series resistors - BOOTSEL and RESET, SWD test points - I2C bus(es) and SPI0/SPI1 pins out to the other sheets"
- company: RoboJackets RoboCup -> (none)
- title: Sensor Suite - MCU -> (none)
