File: pcb/gpio_expander.kicad_sch (KiCad schematic)
At the start: 2 parts

Commit message: add top level schem and cleanup
Parts:
- renumbered R9 to R40, U3 to U7
Other:
- title: IMU Sensor -> GPIO Expander
Changed lines of the file:
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@@
 	(paper "A4")
 	(title_block
-		(title "IMU Sensor")
+		(title "GPIO Expander")
+		(date "2026-10-27")
 	)
 	(rectangle
@@
 	)
 	(hierarchical_label "I2C{SDA,SCL}"
-		(shape output)
+		(shape input)
 		(at 120.65 105.41 180)
 		(effects
@@
 		)
 		(instances
-			(project "GPIO_Expander"
-				(path "/17df1232-b180-49eb-a49c-63e4861e42e5"
+			(project "Onboard_Project"
+				(path "/17df1232-b180-49eb-a49c-63e4861e42e5/e7a9fb03-f871-444e-b288-ebe8cd051421"
 					(reference "#PWR025")
 					(unit 1)
@@
 		(dnp no)
 		(fields_autoplaced yes)
-		(property "Reference" "R9"
+		(property "Reference" "R40"
 			(at 148.59 87.6299 0)
 			(show_name no)
@@
 		)
 		(instances
-			(project "GPIO_Expander"
-				(path "/17df1232-b180-49eb-a49c-63e4861e42e5"
-					(reference "R9")
+			(project "Onboard_Project"
+				(path "/17df1232-b180-49eb-a49c-63e4861e42e5/e7a9fb03-f871-444e-b288-ebe8cd051421"
+					(reference "R40")
 					(unit 1)
 				)
@@
 		)
 		(instances
-			(project "GPIO_Expander"
-				(path "/17df1232-b180-49eb-a49c-63e4861e42e5"
+			(project "Onboard_Project"
+				(path "/17df1232-b180-49eb-a49c-63e4861e42e5/e7a9fb03-f871-444e-b288-ebe8cd051421"
 					(reference "#PWR027")
 					(unit 1)
@@
 		)
 		(instances
-			(project "GPIO_Expander"
-				(path "/17df1232-b180-49eb-a49c-63e4861e42e5"
+			(project "Onboard_Project"
+				(path "/17df1232-b180-49eb-a49c-63e4861e42e5/e7a9fb03-f871-444e-b288-ebe8cd051421"
 					(reference "#PWR026")
 					(unit 1)
@@
 		(dnp no)
 		(fields_autoplaced yes)
-		(property "Reference" "U3"
+		(property "Reference" "U7"
 			(at 163.83 113.03 0)
 			(hide yes)
@@
 		)
 		(instances
-			(project "GPIO_Expander"
-				(path "/17df1232-b180-49eb-a49c-63e4861e42e5"
-					(reference "U3")
+			(project "Onboard_Project"
+				(path "/17df1232-b180-49eb-a49c-63e4861e42e5/e7a9fb03-f871-444e-b288-ebe8cd051421"
+					(reference "U7")
 					(unit 1)
 				)
@@
 		)
 		(instances
-			(project "GPIO_Expander"
-				(path "/17df1232-b180-49eb-a49c-63e4861e42e5"
+			(project "Onboard_Project"
+				(path "/17df1232-b180-49eb-a49c-63e4861e42e5/e7a9fb03-f871-444e-b288-ebe8cd051421"
 					(reference "#PWR024")
 					(unit 1)
@@
 		)
 	)
-	(sheet_instances
-		(path "/"
-			(page "2")
-		)
-	)
-	(embedded_fonts no)
 )

Commit message: cleanup routing
Connections:
- no-connect marks 1 -> 0
Changed lines of the file:
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@@
 		(color 0 0 0 0)
-	)
-	(junction
-		(at 146.05 107.95)
-		(diameter 0)
-		(color 0 0 0 0)
-	)
-	(no_connect
-		(at 140.97 107.95)
 	)
 	(bus_entry
@@
 		)
 		(stroke
-			(width 0)
-			(type default)
-		)
-	)
-	(wire
-		(pts
-			(xy 140.97 107.95) (xy 146.05 107.95)
-		)
-		(stroke

Commit message: Adding docs for GPIO and Color and removing INT
Other:
- moved on the sheet: R40
