File: pcb/Onboard_Project/GPIO_Expander.kicad_sch (KiCad schematic)
At the start: 4 parts

Commit message: move i2c pullup resistors to top schematic
Parts:
- removed R7, R8: 2k, Package_DIP:DIP-8_W7.62mm, symbol Device:R
