File: pcb/Onboard_Project/Onboard_Project_1.kicad_sch (KiCad schematic)
At the start: 25 parts, among them SW1 PTS810, SW2 PTS810, U1 RP2040, U2 W25Q16JVSS, Y1 ABM8-272-T3

Commit message: fix top schematic
Parts:
- added R7, R8: 2k, Resistor_SMD:R_0402_1005Metric, symbol Device:R
Connections:
- net +3.3V: now also R7.1, R8.1
- net I2C.SCL: now also R8.2
- net I2C.SDA: now also R7.2
