File: pcb/Onboard_Project/IMU_Sensor.kicad_sch (KiCad schematic)
At the start: 6 parts

Commit message: move i2c pullup resistors to top schematic
Parts:
- removed R24, R25: 10k, Resistor_SMD:R_0402_1005Metric, symbol Device:R

Commit message: Updating names
Other:
- note added: "Kevin"
Changed lines of the file:
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@@
 	(title_block
 		(title "IMU Sensor")
+		(date "2026-10-27")
+		(rev "Rev 1")
 	)
 	(rectangle
@@
 		)
 	)
+	(text "Kevin"
+		(exclude_from_sim no)
+		(at 184.912 171.704 0)
+		(effects
+			(font
+				(size 1.27 1.27)
+			)
+		)
+	)
