File: pcb/Onboard_Project/led_controller.kicad_sch (KiCad schematic)
At the start: 40 parts, among them IC1 IS31FL3254-QFLS4-TR

Commit message: move i2c pullup resistors to top schematic
Parts:
- removed R12, R13: 2k, Resistor_SMD:R_0402_1005Metric, symbol Device:R

Commit message: Updating names
Other:
- note added: "Madison"
- title: (none) -> LED Controller
Changed lines of the file:
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@@
 	(generator_version "10.0")
 	(paper "A4")
+	(title_block
+		(title "LED Controller")
+		(date "2026-10-27")
+		(rev "Rev 1")
+	)
+	(text "Madison"
+		(exclude_from_sim no)
+		(at 186.436 171.958 0)
+		(effects
+			(font
+				(size 1.27 1.27)
+			)
+		)
+	)
 	(junction
 		(at 143.51 63.5)
@@
 		)
 	)
+	(embedded_fonts no)
 )
